File: hardware/minisumo.kicad_pcb (KiCad board)
At the start: 4 copper layers, 94 x 50 mm, 95 parts, among them J1 MOTOR_L, J2 MOTOR_R, J4 Battery, J5 REMOTE, J6 OLED, Q2 AONR21357, Q3 AO3401A, Q5 AONR21357, SW1 ON_OFF, SW3 BTN_0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

Commit message: ordered
Parts:
- added R18: 330R, Resistor_SMD:R_0402_1005Metric, F.Cu at (59.8, 83.9)
Connections:
- J5 pad 3: /DBG_0 -> /START
Routing:
- net /DBG_0: track 73.7 -> 57.5 mm
- net /START: track 0.00 -> 15.2 mm
- net /BIN1: track 24.5 -> 23.5 mm
- net /AIN1: track 17.5 -> 16.7 mm
- net /BIN2: track 21.4 -> 20.8 mm
- net GND: track 47.5 -> 47.9 mm, vias 116 -> 221
Other:
- board text added: "START"
