File: hardware/motors.kicad_sch (KiCad schematic)
At the start: 27 parts, among them J1 MOTOR_L, J2 MOTOR_R, U1 DRV8848, U13 INA180A2, U14 INA180A2

Commit message: ordered
Other:
- title: (none) -> LOREM
Changed lines of the file:
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@@
 	(generator_version "10.0")
 	(paper "A4")
+	(title_block
+		(title "LOREM")
+		(date "2026-04-06")
+		(rev "1.0")
+	)
 	(junction
 		(at 162.56 100.33)
