File: hardware/power.kicad_sch (KiCad schematic)
At the start: 15 parts, among them J4 Battery, Q2 AONR21357, Q5 AONR21357, SW1 ON_OFF, U2 LMR50410

Commit message: ordered
Other:
- title: (none) -> LOREM
Changed lines of the file:
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@@
 	(generator_version "10.0")
 	(paper "A4")
+	(title_block
+		(title "LOREM")
+		(date "2026-04-06")
+		(rev "1.0")
+	)
 	(text "R_{FBT}/R_{RBB}+V_{REF}=V_{OUT}\n100/24+1=5.17"
 		(exclude_from_sim no)
