File: hardware/sensors.kicad_sch (KiCad schematic)
At the start: 33 parts, among them U10 ITR8307-S17-TR8, U11 LIS3DH, U12 LM393, U15 ITR8307-S17-TR8, U16 ITR8307-S17-TR8, U3 VL53L0X, U4 ITR8307-S17-TR8, U5 VL53L0X, U6 VL53L0X, U7 VL53L0X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

Commit message: ordered
Other:
- title: (none) -> LOREM
Changed lines of the file:
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@@
 	(generator_version "10.0")
 	(paper "A4")
+	(title_block
+		(title "LOREM")
+		(date "2026-04-06")
+		(rev "1.0")
+	)
 	(text "RC filter\n\nPWM TO DAC"
 		(exclude_from_sim no)
