File: hardware/user.kicad_sch (KiCad schematic)
At the start: 14 parts, among them J5 REMOTE, J6 OLED, SW3 BTN_0, SW4 BTN_1

Commit message: ordered
Other:
- note removed: "SPRAWDZ PINOUT!!!!"
- title: (none) -> LOREM
Changed lines of the file:
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@@
 	(generator_version "10.0")
 	(paper "A4")
-	(text "SPRAWDZ PINOUT!!!!"
-		(exclude_from_sim no)
-		(at 162.56 100.838 0)
-		(effects
-			(font
-				(size 1.27 1.27)
-			)
-		)
+	(title_block
+		(title "LOREM")
+		(date "2026-04-06")
+		(rev "1.0")
 	)
 	(junction
